File: hardware/electronic_load.sch (KiCad schematic (older format))
At the start: 27 parts, among them J1 Screw_Terminal_01x02, J2 SPI, J3 UART, P1 Power connector, P2 LCD, P3 One Wire, SW2 Back, SW3 Down, SW4 Up, SW5 Enter, U8 FDV303N

Commit message: Blebleble
Parts:
- added P5, P6: One Wire, Connectors_JST:JST_XH_B03B-XH-A_03x2.50mm_Straight, symbol conn:CONN_01X03
Connections:
- net 3.3V: now also P5.3 (P3), P6.3 (P3)
- net GND: now also J1.2 (Pin_2), P5.1 (P1), P6.1 (P1); no longer J1.1 (Pin_1)
- net ONE_WIRE: now also P5.2 (P2), P6.2 (P2)
- net Variable Load/Vload: now also J1.1 (Pin_1); no longer J1.2 (Pin_2)
Other:
- moved on the sheet: C19, C20, C21, D7, H1, H2, H3, H4, H5, H6, H7, H8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

Commit message: Updates
Connections:
- net GND: now also J1.1 (Pin_1); no longer J1.2 (Pin_2)
- net Variable Load/Vload: now also J1.2 (Pin_2); no longer J1.1 (Pin_1)
Changed lines of the file:
@@
-$EndComp
-$Comp
-L Connector:Screw_Terminal_01x02 J1
-U 1 1 5E987F12
-P 8850 1500
-F 0 "J1" H 8930 1492 50  0000 L CNN
-F 1 "Screw_Terminal_01x02" H 8930 1401 50  0000 L CNN
-F 2 "TerminalBlock_Phoenix:TerminalBlock_Phoenix_MKDS-1,5-2-5.08_1x02_P5.08mm_Horizontal" H 8850 1500 50  0001 C CNN
-F 3 "~" H 8850 1500 50  0001 C CNN
-	1    8850 1500
-	1    0    0    -1
 $EndComp
 $Comp
@@
 	4200 6450 4400 6450
 Connection ~ 4200 5750
+$Comp
+L Connector:Screw_Terminal_01x02 J1
+U 1 1 5E987F12
+P 8850 1600
+F 0 "J1" H 8930 1592 50  0000 L CNN
+F 1 "Screw_Terminal_01x02" H 8930 1501 50  0000 L CNN
+F 2 "TerminalBlock_Phoenix:TerminalBlock_Phoenix_MKDS-1,5-2-5.08_1x02_P5.08mm_Horizontal" H 8850 1600 50  0001 C CNN
+F 3 "~" H 8850 1600 50  0001 C CNN
+	1    8850 1600
+	1    0    0    1
+$EndComp
 $EndSCHEMATC
