File: hardware/electronic_load.kicad_pcb (KiCad board)
At the start: 2 copper layers, 76.8 x 61 mm, 85 parts, among them J1 Screw_Terminal_01x02, J2 SPI, J3 UART, P1 Power connector, P2 LCD, P3 One Wire, P4 Gate Drain Source, SW1 Reset, SW2 Back, SW3 Down, SW4 Up, SW5 Enter, U1 FDV303N, U2 TLV1117-33, U3 LM358, U4 MCP6002-xSN, U5 ATmega1284P-AU, U6 FDV303N, U7 FDV303N, U8 FDV303N, Y1 16MHz

Commit message: Blebleble
Parts:
- added P5: One Wire, Connectors_JST:JST_XH_B03B-XH-A_03x2.50mm_Straight, F.Cu at (111.0, 106.2)
- added P6: One Wire, Connectors_JST:JST_XH_B03B-XH-A_03x2.50mm_Straight, F.Cu at (111.0, 117.3)
- P4: value Gate Drain Source -> CONN_01X03
- moved J1 37.9 mm to (76.0, 76.8), turned to 0 degrees
- moved R3 35.8 mm to (85.6, 73.7), turned to 270 degrees
- moved LS1 32.5 mm to (97.7, 75.3), turned to 180 degrees
- moved C20 31.8 mm to (97.7, 78.2), turned to 270 degrees
- moved R4 31.1 mm to (85.6, 77.0), turned to 270 degrees
- moved D7 29.3 mm to (86.3, 80.8)
- moved C21 27.8 mm to (100.3, 81.1), turned to 270 degrees
- moved R19 24.7 mm to (103.1, 76.5), turned to 0 degrees
- moved U8 24.0 mm to (103.1, 79.2), turned to 0 degrees
- moved P3 23.4 mm to (111.0, 95.0), turned to 90 degrees
- moved R10 20.5 mm to (75.8, 84.0)
- moved P4 15.6 mm to (69.8, 76.1)
- moved H6 8.99 mm to (109.9, 72.6)
- moved H8 8.25 mm to (109.9, 127.0)
- moved H5 3.56 mm to (51.4, 72.6)
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Connections:
- J1 pad 1: GND -> /Variable Load/Vload
- J1 pad 2: /Variable Load/Vload -> GND
Routing:
- net /Variable Load/Vload: track 128.1 -> 47.3 mm
- net 3.3V: track 199.9 -> 227.2 mm, vias 10 -> 9
- net ONE_WIRE: track 62.5 -> 89.3 mm, vias 2 -> 3
- net /Variable Load/Current_feedback_P: track 39.7 -> 61.3 mm, vias 12 -> 0
- net VOLTAGE_SENSE: track 57.4 -> 75.4 mm
- net (no net): track 28.3 -> 39.9 mm, vias 4 -> 2
- net Net-(P4-Pad3): track 43.5 -> 54.4 mm, vias 2 -> 3
- net GND: track 59.9 -> 52.1 mm, vias 32 -> 28
- net SPEAKER_DRIVE: track 78.3 -> 76.4 mm, vias 3 -> 4
- net 12V: track 44.3 -> 45.2 mm
Other:
- board size 76.8 x 61 mm -> 68.6 x 64.5 mm

Commit message: Fixup
Parts:
- C16, C5: moved to B.Cu
- moved C5 6.10 mm to (86.4, 106.7), turned to 90 degrees
- moved C16 5.62 mm to (86.4, 97.0), turned to 90 degrees
- moved D8 1.36 mm to (90.7, 115.7)
- moved R24 1.08 mm to (90.6, 112.9)
- moved C14 0.89 mm to (87.0, 112.9)
- moved R25 0.83 mm to (87.1, 115.1)
- moved R9 0.52 mm to (90.3, 110.7), turned to 180 degrees
- moved R13 0.51 mm to (87.0, 110.7)
Routing:
- net GND: track 52.1 -> 58.3 mm, vias 28 -> 24
- net 3.3V: track 227.2 -> 230.3 mm, vias 9 -> 10
- net VOLTAGE_SENSE: track 75.4 -> 78.5 mm
- net 12V: track 45.2 -> 47.8 mm, vias 1 -> 2
- net Net-(C1-Pad2): track 21.6 -> 19.9 mm
- net CURRENT_SENSE: track 11.1 -> 9.85 mm
- net Net-(C14-Pad1): track 11.2 -> 10.3 mm

Commit message: Updates
Parts:
- moved J1 5.17 mm to (81.2, 76.1), turned to 180 degrees
Connections:
- J1 pad 1: /Variable Load/Vload -> GND
- J1 pad 2: GND -> /Variable Load/Vload
Routing:
- net Net-(D8-Pad1): track 34.5 -> 35.4 mm
- net 3.3V: track 230.3 -> 231.2 mm
- net /Variable Load/Enable_inv: track 39.8 -> 40.4 mm
- net VOLTAGE_SENSE: track 78.5 -> 79.0 mm

Commit message: Fixes
Parts:
- P4: value CONN_01X03 -> Gate Drain Source
Changed lines of the file:
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@@
     (add_net "Net-(C21-Pad1)")
     (add_net "Net-(D1-Pad1)")
-    (add_net "Net-(D1-Pad2)")
     (add_net "Net-(D3-Pad1)")
     (add_net "Net-(D4-Pad1)")
@@
     (add_net "Net-(U3-Pad6)")
     (add_net "Net-(U4-Pad6)")
-    (add_net "Net-(U5-Pad11)")
-    (add_net "Net-(U5-Pad12)")
-    (add_net "Net-(U5-Pad16)")
-    (add_net "Net-(U5-Pad30)")
-    (add_net "Net-(U5-Pad31)")
-    (add_net "Net-(U5-Pad32)")
-    (add_net "Net-(U5-Pad34)")
-    (add_net "Net-(U5-Pad35)")
-    (add_net "Net-(U5-Pad40)")
-    (add_net "Net-(U5-Pad41)")
-    (add_net "Net-(U5-Pad42)")
-    (add_net "Net-(U5-Pad43)")
     (add_net ONE_WIRE)
     (add_net SCL)
@@
       (effects (font (size 1 1) (thickness 0.15)))
     )
-    (fp_text value CONN_01X03 (at 5.2832 6.0452) (layer F.SilkS)
+    (fp_text value "Gate Drain Source" (at 5.2197 6.4262) (layer F.SilkS)
       (effects (font (size 1 1) (thickness 0.15)))
     )
@@
     (fp_line (start 8.13 5.1) (end 8.13 -5.71) (layer F.CrtYd) (width 0.05))
     (fp_line (start 8.13 -5.71) (end -3.04 -5.71) (layer F.CrtYd) (width 0.05))
-    (fp_text user "LOAD+ LOAD-" (at 2.7178 -6.6802) (layer F.SilkS)
-      (effects (font (size 1 1) (thickness 0.15)))
-    )
+    (fp_text user "LOAD+ LOAD-" (at 1.9685 6.2865) (layer F.SilkS)
+      (effects (font (size 1 1) (thickness 0.15)))
+    )

Commit message: First commit of code
Routing:
- net GND: vias 24 -> 25
- net /Variable Load/Current_feedback_P: vias 0 -> 12
- net (no net): vias 2 -> 3
Other:
- board text added: "Design by Daniel Karling 2020"
