File: hardware/load.sch (KiCad schematic (older format))
At the start: 25 parts, among them P4 CONN_01X03, U1 FDV303N, U3 LM358, U4 MCP6002-xSN, U6 FDV303N, U7 FDV303N

Commit message: First commit of code
Connections:
- net Current_feedback_N is gone; now on net GND: R14.2
Changed lines of the file:
@@
 Wire Wire Line
 	7300 3200 7300 3850
-Wire Wire Line
-	7750 3150 7750 3300
 $Comp
 L Device:R R17
@@
 Wire Wire Line
 	7300 1850 7300 2050
+Wire Wire Line
+	7750 3150 7750 3200
+Wire Wire Line
+	7300 3200 7750 3200
+Connection ~ 7750 3200
+Wire Wire Line
+	7750 3200 7750 3300
 $EndSCHEMATC
